File: KeebPcb/_autosave-KeebPcb.kicad_pcb (KiCad board)
At the start: 2 copper layers, 89.6 x 38.1 mm, 25 parts, among them SW1 SW_Push, U1 ATmega32U4-A, Y1 16MHz

Commit message: Full Design done Pending like changing to USB-C and adding LED
Parts:
- removed G***: LOGO, Photo:Untitled
Routing:
- net GND: track 126.7 -> 158.1 mm
Other:
- board size 89.6 x 38.1 mm -> 91.1 x 38.1 mm
